File: TKD_PCB/ledring.sch (KiCad schematic (older format))
At the start: 48 parts

Commit message: Begin of the final assembly
Parts:
- C14, C17, C20, C23, C26: renamed from C?; footprint (none) -> Capacitor_SMD:C_0805_2012Metric
- gave numbers to parts that had none: 43

Commit message: did Remco's homework
Parts:
- C14: footprint Capacitor_SMD:C_0805_2012Metric -> Capacitor_SMD:C_0805_2012Metric_Pad1.15x1.40mm_HandSolder; LCSC (none) -> C354369
- C15: renamed from C17; footprint Capacitor_SMD:C_0805_2012Metric -> Capacitor_SMD:C_0805_2012Metric_Pad1.15x1.40mm_HandSolder; LCSC (none) -> C354369
- C16: renamed from C20; footprint Capacitor_SMD:C_0805_2012Metric -> Capacitor_SMD:C_0805_2012Metric_Pad1.15x1.40mm_HandSolder; LCSC (none) -> C354369
- C17: renamed from C23; footprint Capacitor_SMD:C_0805_2012Metric -> Capacitor_SMD:C_0805_2012Metric_Pad1.15x1.40mm_HandSolder; LCSC (none) -> C354369
- C18: renamed from C26; footprint Capacitor_SMD:C_0805_2012Metric -> Capacitor_SMD:C_0805_2012Metric_Pad1.15x1.40mm_HandSolder; LCSC (none) -> C354369
- C19: renamed from C29; footprint (none) -> Capacitor_SMD:C_0805_2012Metric_Pad1.15x1.40mm_HandSolder; LCSC (none) -> C354369
- C20: renamed from C32; footprint (none) -> Capacitor_SMD:C_0805_2012Metric_Pad1.15x1.40mm_HandSolder; LCSC (none) -> C354369
- C21: renamed from C35; footprint (none) -> Capacitor_SMD:C_0805_2012Metric_Pad1.15x1.40mm_HandSolder; LCSC (none) -> C354369
- C22: renamed from C15; footprint (none) -> Capacitor_SMD:C_0805_2012Metric_Pad1.15x1.40mm_HandSolder; LCSC (none) -> C354369
- C23: renamed from C18; footprint (none) -> Capacitor_SMD:C_0805_2012Metric_Pad1.15x1.40mm_HandSolder; LCSC (none) -> C354369
- C24: renamed from C21; footprint (none) -> Capacitor_SMD:C_0805_2012Metric_Pad1.15x1.40mm_HandSolder; LCSC (none) -> C354369
- C25: renamed from C24; footprint (none) -> Capacitor_SMD:C_0805_2012Metric_Pad1.15x1.40mm_HandSolder; LCSC (none) -> C354369
- C26: renamed from C27; footprint (none) -> Capacitor_SMD:C_0805_2012Metric_Pad1.15x1.40mm_HandSolder; LCSC (none) -> C354369
- C27: renamed from C30; footprint (none) -> Capacitor_SMD:C_0805_2012Metric_Pad1.15x1.40mm_HandSolder; LCSC (none) -> C354369
- C28: renamed from C33; footprint (none) -> Capacitor_SMD:C_0805_2012Metric_Pad1.15x1.40mm_HandSolder; LCSC (none) -> C354369
- C29: renamed from C36; footprint (none) -> Capacitor_SMD:C_0805_2012Metric_Pad1.15x1.40mm_HandSolder; LCSC (none) -> C354369
- C30: renamed from C16; footprint (none) -> Capacitor_SMD:C_0805_2012Metric_Pad1.15x1.40mm_HandSolder; LCSC (none) -> C354369
- C31: renamed from C19; footprint (none) -> Capacitor_SMD:C_0805_2012Metric_Pad1.15x1.40mm_HandSolder; LCSC (none) -> C354369
- C32: renamed from C22; footprint (none) -> Capacitor_SMD:C_0805_2012Metric_Pad1.15x1.40mm_HandSolder; LCSC (none) -> C354369
- C33: renamed from C25; footprint (none) -> Capacitor_SMD:C_0805_2012Metric_Pad1.15x1.40mm_HandSolder; LCSC (none) -> C354369
- C34: renamed from C28; footprint (none) -> Capacitor_SMD:C_0805_2012Metric_Pad1.15x1.40mm_HandSolder; LCSC (none) -> C354369
- C35: renamed from C31; footprint (none) -> Capacitor_SMD:C_0805_2012Metric_Pad1.15x1.40mm_HandSolder; LCSC (none) -> C354369
- C36: renamed from C34; footprint (none) -> Capacitor_SMD:C_0805_2012Metric_Pad1.15x1.40mm_HandSolder; LCSC (none) -> C354369
- C37: footprint (none) -> Capacitor_SMD:C_0805_2012Metric_Pad1.15x1.40mm_HandSolder; LCSC (none) -> C354369
- D10: renamed from D16; LCSC (none) -> C114586
- D11: renamed from D19; LCSC (none) -> C114586
- D12: renamed from D22; LCSC (none) -> C114586
- D13: renamed from D25; LCSC (none) -> C114586
- D14: renamed from D28; LCSC (none) -> C114586
- D15: renamed from D8; LCSC (none) -> C114586
- D16: renamed from D11; LCSC (none) -> C114586
- D17: renamed from D14; LCSC (none) -> C114586
- D18: renamed from D17; LCSC (none) -> C114586
- D19: renamed from D20; LCSC (none) -> C114586
- D20: renamed from D23; LCSC (none) -> C114586
- D21: renamed from D26; LCSC (none) -> C114586
- D22: renamed from D29; LCSC (none) -> C114586
- D23: renamed from D9; LCSC (none) -> C114586
- D24: renamed from D12; LCSC (none) -> C114586
- D25: renamed from D15; LCSC (none) -> C114586
- D26: renamed from D18; LCSC (none) -> C114586
- D27: renamed from D21; LCSC (none) -> C114586
- D28: renamed from D24; LCSC (none) -> C114586
- D29: renamed from D27; LCSC (none) -> C114586
- D30, D7: LCSC (none) -> C114586
- D8: renamed from D10; LCSC (none) -> C114586
- D9: renamed from D13; LCSC (none) -> C114586; LSCS (none) -> C114586
